Commit message: sync: 2026-10-21 20:50:15 +0800

File: modules/wheeled_description/wheeled_arm_v2/urdf/wheeled_arm_v2.urdf (robot description, URDF)
Before this commit: robot wheeled_arm_v2, 13 links, 12 joints
Joints:
- joint Arm_P1: limit lower=-1.57 upper=1.57 effort=9 velocity=0 -> lower=-1.57 upper=1.57 effort=27 velocity=0
- joint Arm_P2: limit lower=-1.57 upper=1.57 effort=9 velocity=0 -> lower=-1.57 upper=1.57 effort=27 velocity=0
- joint Arm_R: limit lower=-3.14 upper=3.14 effort=9 velocity=0 -> lower=-3.14 upper=3.14 effort=27 velocity=0
- joint Arm_Y1: limit lower=-1.57 upper=1.57 effort=9 velocity=0 -> lower=-1.57 upper=1.57 effort=27 velocity=0
- joint Arm_Y2: limit lower=-1.57 upper=1.57 effort=9 velocity=0 -> lower=-1.57 upper=1.57 effort=27 velocity=0
- joint Arm_Y3: limit lower=-1.57 upper=1.57 effort=9 velocity=0 -> lower=-1.57 upper=1.57 effort=27 velocity=0
- joint HubL: limit effort=9.6 velocity=115 -> effort=17 velocity=115
- joint HubR: limit effort=9.6 velocity=115 -> effort=17 velocity=115

File: modules/wheeled_description/wheeled_leg_v2/urdf/wheeled_leg_v2.urdf (robot description, URDF)
Before this commit: robot wheeled_leg_v2, 7 links, 6 joints
Joints:
- joint HubL: limit effort=9.6 velocity=115 -> effort=17 velocity=115
- joint HubR: limit effort=9.6 velocity=115 -> effort=17 velocity=115
